Commit message: [ADD] pose-publisher for actor

File: config/skins/BrownShirtGuyMoonwalk/model.sdf.xacro (robot description, xacro)
@@ -19,5 +19,5 @@
   <xacro:property name="vel_topic"  value="${ns}/cmd_vel" />
   <xacro:property name="path_topic" value="${ns}/cmd_path" />
-  <!-- SDF output -->
+  <xacro:property name="pose_topic" value="${ns}/pose" />
   <actor name="$(arg actor_name)">
     <skin>
@@ -30,10 +30,9 @@
       <interpolate_x>true</interpolate_x>
     </animation>
-    <plugin filename="libgazebo_ros_actor_plugin.so"
-            name="gazebo_ros_actor_plugin::GazeboRosActorCommand">
+    <plugin filename="libgazebo_ros_actor_plugin.so" name="gazebo_ros_actor_plugin::GazeboRosActorCommand">
       <follow_mode>$(arg follow_mode)</follow_mode>
       <vel_topic>${vel_topic}</vel_topic>
       <path_topic>${path_topic}</path_topic>
-      <animation_factor>2.5</animation_factor>
+      <animation_factor>1.0</animation_factor>
       <linear_tolerance>0.1</linear_tolerance>
       <linear_velocity>$(arg linear_velocity)</linear_velocity>
@@ -41,4 +40,7 @@
       <angular_velocity>2.5</angular_velocity>
       <default_rotation>1.57</default_rotation>
+      <pose_topic>${pose_topic}</pose_topic>
+      <publish_pose>true</publish_pose>
+      <pose_publish_rate>30</pose_publish_rate>
     </plugin>
   </actor>

File: config/skins/DoctorFemaleWalk/model.sdf.xacro (robot description, xacro)
@@ -19,5 +19,5 @@
   <xacro:property name="vel_topic"  value="${ns}/cmd_vel" />
   <xacro:property name="path_topic" value="${ns}/cmd_path" />
-  <!-- SDF output -->
+  <xacro:property name="pose_topic" value="${ns}/pose" />
   <actor name="$(arg actor_name)">
     <skin>
@@ -30,6 +30,5 @@
       <interpolate_x>true</interpolate_x>
     </animation>
-    <plugin filename="libgazebo_ros_actor_plugin.so"
-            name="gazebo_ros_actor_plugin::GazeboRosActorCommand">
+    <plugin filename="libgazebo_ros_actor_plugin.so" name="gazebo_ros_actor_plugin::GazeboRosActorCommand">
       <follow_mode>$(arg follow_mode)</follow_mode>
       <vel_topic>${vel_topic}</vel_topic>
@@ -41,4 +40,7 @@
       <angular_velocity>2.5</angular_velocity>
       <default_rotation>1.57</default_rotation>
+      <pose_topic>${pose_topic}</pose_topic>
+      <publish_pose>true</publish_pose>
+      <pose_publish_rate>30</pose_publish_rate>
     </plugin>
   </actor>

File: config/skins/GreenShirtGuy/model.sdf.xacro (robot description, xacro)
@@ -19,5 +19,5 @@
   <xacro:property name="vel_topic"  value="${ns}/cmd_vel" />
   <xacro:property name="path_topic" value="${ns}/cmd_path" />
-  <!-- SDF output -->
+  <xacro:property name="pose_topic" value="${ns}/pose" />
   <actor name="$(arg actor_name)">
     <skin>
@@ -30,10 +30,9 @@
       <interpolate_x>true</interpolate_x>
     </animation>
-    <plugin filename="libgazebo_ros_actor_plugin.so"
-            name="gazebo_ros_actor_plugin::GazeboRosActorCommand">
+    <plugin filename="libgazebo_ros_actor_plugin.so" name="gazebo_ros_actor_plugin::GazeboRosActorCommand">
       <follow_mode>$(arg follow_mode)</follow_mode>
       <vel_topic>${vel_topic}</vel_topic>
       <path_topic>${path_topic}</path_topic>
-      <animation_factor>2.5</animation_factor>
+      <animation_factor>1.0</animation_factor>
       <linear_tolerance>0.1</linear_tolerance>
       <linear_velocity>$(arg linear_velocity)</linear_velocity>
@@ -41,4 +40,7 @@
       <angular_velocity>2.5</angular_velocity>
       <default_rotation>1.57</default_rotation>
+      <pose_topic>${pose_topic}</pose_topic>
+      <publish_pose>true</publish_pose>
+      <pose_publish_rate>30</pose_publish_rate>
     </plugin>
   </actor>

File: config/skins/GreenShirtGuyRunning/model.sdf.xacro (robot description, xacro)
@@ -19,5 +19,5 @@
   <xacro:property name="vel_topic"  value="${ns}/cmd_vel" />
   <xacro:property name="path_topic" value="${ns}/cmd_path" />
-  <!-- SDF output -->
+  <xacro:property name="pose_topic" value="${ns}/pose" />
   <actor name="$(arg actor_name)">
     <skin>
@@ -30,6 +30,5 @@
       <interpolate_x>true</interpolate_x>
     </animation>
-    <plugin filename="libgazebo_ros_actor_plugin.so"
-            name="gazebo_ros_actor_plugin::GazeboRosActorCommand">
+    <plugin filename="libgazebo_ros_actor_plugin.so" name="gazebo_ros_actor_plugin::GazeboRosActorCommand">
       <follow_mode>$(arg follow_mode)</follow_mode>
       <vel_topic>${vel_topic}</vel_topic>
@@ -41,4 +40,7 @@
       <angular_velocity>2.5</angular_velocity>
       <default_rotation>1.57</default_rotation>
+      <pose_topic>${pose_topic}</pose_topic>
+      <publish_pose>true</publish_pose>
+      <pose_publish_rate>30</pose_publish_rate>
     </plugin>
   </actor>

Commit message: [FIX] publish_pose is both launch-argument and xacro argument

File: config/skins/BrownShirtGuyMoonwalk/model.sdf.xacro (robot description, xacro)
@@ -6,4 +6,5 @@
   <xacro:arg name="follow_mode" default="velocity"/>
   <xacro:arg name="linear_velocity" default="1.0"/>
+  <xacro:arg name="publish_pose" default="true"/>
   <!-- Validate follow_mode -->
   <xacro:if value="${'$(arg follow_mode)' != 'velocity' and '$(arg follow_mode)' != 'path'}">
@@ -15,4 +16,5 @@
   <xacro:property name="prefix" value="$(arg gazebo_topic_prefix)"/>
   <xacro:property name="name"   value="$(arg actor_name)"/>
+  <xacro:property name="publishpose" value="$(arg publish_pose)"/>
   <!-- Clean namespace handling -->
   <xacro:property name="ns" value="${prefix + '/' if prefix else ''}${name}" />
@@ -41,5 +43,5 @@
       <default_rotation>1.57</default_rotation>
       <pose_topic>${pose_topic}</pose_topic>
-      <publish_pose>true</publish_pose>
+      <publish_pose>${publishpose}</publish_pose>
       <pose_publish_rate>30</pose_publish_rate>
     </plugin>

File: config/skins/DoctorFemaleWalk/model.sdf.xacro (robot description, xacro)
@@ -6,4 +6,5 @@
   <xacro:arg name="follow_mode" default="velocity"/>
   <xacro:arg name="linear_velocity" default="1.0"/>
+  <xacro:arg name="publish_pose" default="true"/>
   <!-- Validate follow_mode -->
   <xacro:if value="${'$(arg follow_mode)' != 'velocity' and '$(arg follow_mode)' != 'path'}">
@@ -15,4 +16,5 @@
   <xacro:property name="prefix" value="$(arg gazebo_topic_prefix)"/>
   <xacro:property name="name"   value="$(arg actor_name)"/>
+  <xacro:property name="publishpose" value="$(arg publish_pose)"/>
   <!-- Clean namespace handling -->
   <xacro:property name="ns" value="${prefix + '/' if prefix else ''}${name}" />
@@ -41,5 +43,5 @@
       <default_rotation>1.57</default_rotation>
       <pose_topic>${pose_topic}</pose_topic>
-      <publish_pose>true</publish_pose>
+      <publish_pose>${publishpose}</publish_pose>
       <pose_publish_rate>30</pose_publish_rate>
     </plugin>

File: config/skins/GreenShirtGuy/model.sdf.xacro (robot description, xacro)
@@ -6,4 +6,5 @@
   <xacro:arg name="follow_mode" default="velocity"/>
   <xacro:arg name="linear_velocity" default="1.0"/>
+  <xacro:arg name="publish_pose" default="true"/>
   <!-- Validate follow_mode -->
   <xacro:if value="${'$(arg follow_mode)' != 'velocity' and '$(arg follow_mode)' != 'path'}">
@@ -15,4 +16,5 @@
   <xacro:property name="prefix" value="$(arg gazebo_topic_prefix)"/>
   <xacro:property name="name"   value="$(arg actor_name)"/>
+  <xacro:property name="publishpose" value="$(arg publish_pose)"/>
   <!-- Clean namespace handling -->
   <xacro:property name="ns" value="${prefix + '/' if prefix else ''}${name}" />
@@ -41,5 +43,5 @@
       <default_rotation>1.57</default_rotation>
       <pose_topic>${pose_topic}</pose_topic>
-      <publish_pose>true</publish_pose>
+      <publish_pose>${publishpose}</publish_pose>
       <pose_publish_rate>30</pose_publish_rate>
     </plugin>

File: config/skins/GreenShirtGuyRunning/model.sdf.xacro (robot description, xacro)
@@ -6,4 +6,5 @@
   <xacro:arg name="follow_mode" default="velocity"/>
   <xacro:arg name="linear_velocity" default="3.0"/>
+  <xacro:arg name="publish_pose" default="true"/>
   <!-- Validate follow_mode -->
   <xacro:if value="${'$(arg follow_mode)' != 'velocity' and '$(arg follow_mode)' != 'path'}">
@@ -15,4 +16,5 @@
   <xacro:property name="prefix" value="$(arg gazebo_topic_prefix)"/>
   <xacro:property name="name"   value="$(arg actor_name)"/>
+  <xacro:property name="publishpose" value="$(arg publish_pose)"/>
   <!-- Clean namespace handling -->
   <xacro:property name="ns" value="${prefix + '/' if prefix else ''}${name}" />
@@ -41,5 +43,5 @@
       <default_rotation>1.57</default_rotation>
       <pose_topic>${pose_topic}</pose_topic>
-      <publish_pose>true</publish_pose>
+      <publish_pose>${publishpose}</publish_pose>
       <pose_publish_rate>30</pose_publish_rate>
     </plugin>

Commit message: [ADD] pose publisher with offset

File: config/skins/BrownShirtGuyMoonwalk/model.sdf.xacro (robot description, xacro)
@@ -7,4 +7,11 @@
   <xacro:arg name="linear_velocity" default="1.0"/>
   <xacro:arg name="publish_pose" default="true"/>
+  <xacro:arg name="pose_publish_rate" default="30.0"/>
+  <xacro:arg name="pose_offset_x" default="0.0"/>
+  <xacro:arg name="pose_offset_y" default="0.0"/>
+  <xacro:arg name="pose_offset_z" default="0.0"/>
+  <xacro:arg name="pose_offset_roll" default="0.0"/>
+  <xacro:arg name="pose_offset_pitch" default="0.0"/>
+  <xacro:arg name="pose_offset_yaw" default="0.0"/>
   <!-- Validate follow_mode -->
   <xacro:if value="${'$(arg follow_mode)' != 'velocity' and '$(arg follow_mode)' != 'path'}">
@@ -13,13 +20,20 @@
     </xacro:error>
   </xacro:if>
-  <!-- Clean topic construction using expressions (no nested if/unless inside property) -->
+  <!-- Clean topic construction & handling namespace -->
   <xacro:property name="prefix" value="$(arg gazebo_topic_prefix)"/>
   <xacro:property name="name"   value="$(arg actor_name)"/>
   <xacro:property name="publishpose" value="$(arg publish_pose)"/>
-  <!-- Clean namespace handling -->
   <xacro:property name="ns" value="${prefix + '/' if prefix else ''}${name}" />
   <xacro:property name="vel_topic"  value="${ns}/cmd_vel" />
   <xacro:property name="path_topic" value="${ns}/cmd_path" />
   <xacro:property name="pose_topic" value="${ns}/pose" />
+  <xacro:property name="publish_rate" value="$(arg pose_publish_rate)" />
+  <!-- pose offsets -->
+  <xacro:property name="poseoffset_x" value="$(arg pose_offset_x)" />
+  <xacro:property name="poseoffset_y" value="$(arg pose_offset_y)" />
+  <xacro:property name="poseoffset_z" value="$(arg pose_offset_z)" />
+  <xacro:property name="poseoffset_roll" value="$(arg pose_offset_roll)" />
+  <xacro:property name="poseoffset_pitch" value="$(arg pose_offset_pitch)" />
+  <xacro:property name="poseoffset_yaw" value="$(arg pose_offset_yaw)" />
   <actor name="$(arg actor_name)">
     <skin>
@@ -44,5 +58,11 @@
       <pose_topic>${pose_topic}</pose_topic>
       <publish_pose>${publishpose}</publish_pose>
-      <pose_publish_rate>30</pose_publish_rate>
+      <pose_publish_rate>${publish_rate}</pose_publish_rate>
+      <pose_offset_x>${poseoffset_x}</pose_offset_x>
+      <pose_offset_y>${poseoffset_y}</pose_offset_y>
+      <pose_offset_z>${poseoffset_z}</pose_offset_z>
+      <pose_offset_roll>${poseoffset_roll}</pose_offset_roll>
+      <pose_offset_pitch>${poseoffset_pitch}</pose_offset_pitch>
+      <pose_offset_yaw>${poseoffset_yaw}</pose_offset_yaw>
     </plugin>
   </actor>

File: config/skins/DoctorFemaleWalk/model.sdf.xacro (robot description, xacro)
@@ -7,4 +7,11 @@
   <xacro:arg name="linear_velocity" default="1.0"/>
   <xacro:arg name="publish_pose" default="true"/>
+  <xacro:arg name="pose_publish_rate" default="30.0"/>
+  <xacro:arg name="pose_offset_x" default="0.0"/>
+  <xacro:arg name="pose_offset_y" default="0.0"/>
+  <xacro:arg name="pose_offset_z" default="0.0"/>
+  <xacro:arg name="pose_offset_roll" default="0.0"/>
+  <xacro:arg name="pose_offset_pitch" default="0.0"/>
+  <xacro:arg name="pose_offset_yaw" default="0.0"/>
   <!-- Validate follow_mode -->
   <xacro:if value="${'$(arg follow_mode)' != 'velocity' and '$(arg follow_mode)' != 'path'}">
@@ -13,13 +20,20 @@
     </xacro:error>
   </xacro:if>
-  <!-- Clean topic construction using expressions (no nested if/unless inside property) -->
+  <!-- Clean topic construction & handling namespace -->
   <xacro:property name="prefix" value="$(arg gazebo_topic_prefix)"/>
   <xacro:property name="name"   value="$(arg actor_name)"/>
   <xacro:property name="publishpose" value="$(arg publish_pose)"/>
-  <!-- Clean namespace handling -->
   <xacro:property name="ns" value="${prefix + '/' if prefix else ''}${name}" />
   <xacro:property name="vel_topic"  value="${ns}/cmd_vel" />
   <xacro:property name="path_topic" value="${ns}/cmd_path" />
   <xacro:property name="pose_topic" value="${ns}/pose" />
+  <xacro:property name="publish_rate" value="$(arg pose_publish_rate)" />
+  <!-- pose offsets -->
+  <xacro:property name="poseoffset_x" value="$(arg pose_offset_x)" />
+  <xacro:property name="poseoffset_y" value="$(arg pose_offset_y)" />
+  <xacro:property name="poseoffset_z" value="$(arg pose_offset_z)" />
+  <xacro:property name="poseoffset_roll" value="$(arg pose_offset_roll)" />
+  <xacro:property name="poseoffset_pitch" value="$(arg pose_offset_pitch)" />
+  <xacro:property name="poseoffset_yaw" value="$(arg pose_offset_yaw)" />
   <actor name="$(arg actor_name)">
     <skin>
@@ -44,5 +58,11 @@
       <pose_topic>${pose_topic}</pose_topic>
       <publish_pose>${publishpose}</publish_pose>
-      <pose_publish_rate>30</pose_publish_rate>
+      <pose_publish_rate>${publish_rate}</pose_publish_rate>
+      <pose_offset_x>${poseoffset_x}</pose_offset_x>
+      <pose_offset_y>${poseoffset_y}</pose_offset_y>
+      <pose_offset_z>${poseoffset_z}</pose_offset_z>
+      <pose_offset_roll>${poseoffset_roll}</pose_offset_roll>
+      <pose_offset_pitch>${poseoffset_pitch}</pose_offset_pitch>
+      <pose_offset_yaw>${poseoffset_yaw}</pose_offset_yaw>
     </plugin>
   </actor>

File: config/skins/GreenShirtGuy/model.sdf.xacro (robot description, xacro)
@@ -7,4 +7,11 @@
   <xacro:arg name="linear_velocity" default="1.0"/>
   <xacro:arg name="publish_pose" default="true"/>
+  <xacro:arg name="pose_publish_rate" default="30.0"/>
+  <xacro:arg name="pose_offset_x" default="0.0"/>
+  <xacro:arg name="pose_offset_y" default="0.0"/>
+  <xacro:arg name="pose_offset_z" default="0.0"/>
+  <xacro:arg name="pose_offset_roll" default="0.0"/>
+  <xacro:arg name="pose_offset_pitch" default="0.0"/>
+  <xacro:arg name="pose_offset_yaw" default="0.0"/>
   <!-- Validate follow_mode -->
   <xacro:if value="${'$(arg follow_mode)' != 'velocity' and '$(arg follow_mode)' != 'path'}">
@@ -13,13 +20,20 @@
     </xacro:error>
   </xacro:if>
-  <!-- Clean topic construction using expressions (no nested if/unless inside property) -->
+  <!-- Clean topic construction & handling namespace -->
   <xacro:property name="prefix" value="$(arg gazebo_topic_prefix)"/>
   <xacro:property name="name"   value="$(arg actor_name)"/>
   <xacro:property name="publishpose" value="$(arg publish_pose)"/>
-  <!-- Clean namespace handling -->
   <xacro:property name="ns" value="${prefix + '/' if prefix else ''}${name}" />
   <xacro:property name="vel_topic"  value="${ns}/cmd_vel" />
   <xacro:property name="path_topic" value="${ns}/cmd_path" />
   <xacro:property name="pose_topic" value="${ns}/pose" />
+  <xacro:property name="publish_rate" value="$(arg pose_publish_rate)" />
+  <!-- pose offsets -->
+  <xacro:property name="poseoffset_x" value="$(arg pose_offset_x)" />
+  <xacro:property name="poseoffset_y" value="$(arg pose_offset_y)" />
+  <xacro:property name="poseoffset_z" value="$(arg pose_offset_z)" />
+  <xacro:property name="poseoffset_roll" value="$(arg pose_offset_roll)" />
+  <xacro:property name="poseoffset_pitch" value="$(arg pose_offset_pitch)" />
+  <xacro:property name="poseoffset_yaw" value="$(arg pose_offset_yaw)" />
   <actor name="$(arg actor_name)">
     <skin>
@@ -44,5 +58,11 @@
       <pose_topic>${pose_topic}</pose_topic>
       <publish_pose>${publishpose}</publish_pose>
-      <pose_publish_rate>30</pose_publish_rate>
+      <pose_publish_rate>${publish_rate}</pose_publish_rate>
+      <pose_offset_x>${poseoffset_x}</pose_offset_x>
+      <pose_offset_y>${poseoffset_y}</pose_offset_y>
+      <pose_offset_z>${poseoffset_z}</pose_offset_z>
+      <pose_offset_roll>${poseoffset_roll}</pose_offset_roll>
+      <pose_offset_pitch>${poseoffset_pitch}</pose_offset_pitch>
+      <pose_offset_yaw>${poseoffset_yaw}</pose_offset_yaw>
     </plugin>
   </actor>

File: config/skins/GreenShirtGuyRunning/model.sdf.xacro (robot description, xacro)
@@ -7,4 +7,11 @@
   <xacro:arg name="linear_velocity" default="3.0"/>
   <xacro:arg name="publish_pose" default="true"/>
+  <xacro:arg name="pose_publish_rate" default="30.0"/>
+  <xacro:arg name="pose_offset_x" default="0.0"/>
+  <xacro:arg name="pose_offset_y" default="0.0"/>
+  <xacro:arg name="pose_offset_z" default="0.0"/>
+  <xacro:arg name="pose_offset_roll" default="0.0"/>
+  <xacro:arg name="pose_offset_pitch" default="0.0"/>
+  <xacro:arg name="pose_offset_yaw" default="0.0"/>
   <!-- Validate follow_mode -->
   <xacro:if value="${'$(arg follow_mode)' != 'velocity' and '$(arg follow_mode)' != 'path'}">
@@ -13,13 +20,20 @@
     </xacro:error>
   </xacro:if>
-  <!-- Clean topic construction using expressions (no nested if/unless inside property) -->
+  <!-- Clean topic construction & handling namespace -->
   <xacro:property name="prefix" value="$(arg gazebo_topic_prefix)"/>
   <xacro:property name="name"   value="$(arg actor_name)"/>
   <xacro:property name="publishpose" value="$(arg publish_pose)"/>
-  <!-- Clean namespace handling -->
   <xacro:property name="ns" value="${prefix + '/' if prefix else ''}${name}" />
   <xacro:property name="vel_topic"  value="${ns}/cmd_vel" />
   <xacro:property name="path_topic" value="${ns}/cmd_path" />
   <xacro:property name="pose_topic" value="${ns}/pose" />
+  <xacro:property name="publish_rate" value="$(arg pose_publish_rate)" />
+  <!-- pose offsets -->
+  <xacro:property name="poseoffset_x" value="$(arg pose_offset_x)" />
+  <xacro:property name="poseoffset_y" value="$(arg pose_offset_y)" />
+  <xacro:property name="poseoffset_z" value="$(arg pose_offset_z)" />
+  <xacro:property name="poseoffset_roll" value="$(arg pose_offset_roll)" />
+  <xacro:property name="poseoffset_pitch" value="$(arg pose_offset_pitch)" />
+  <xacro:property name="poseoffset_yaw" value="$(arg pose_offset_yaw)" />
   <actor name="$(arg actor_name)">
     <skin>
@@ -44,5 +58,11 @@
       <pose_topic>${pose_topic}</pose_topic>
       <publish_pose>${publishpose}</publish_pose>
-      <pose_publish_rate>30</pose_publish_rate>
+      <pose_publish_rate>${publish_rate}</pose_publish_rate>
+      <pose_offset_x>${poseoffset_x}</pose_offset_x>
+      <pose_offset_y>${poseoffset_y}</pose_offset_y>
+      <pose_offset_z>${poseoffset_z}</pose_offset_z>
+      <pose_offset_roll>${poseoffset_roll}</pose_offset_roll>
+      <pose_offset_pitch>${poseoffset_pitch}</pose_offset_pitch>
+      <pose_offset_yaw>${poseoffset_yaw}</pose_offset_yaw>
     </plugin>
   </actor>
